Commit message: házban tesztelve, GAZEBO jó, RVIZ+SLAM is jobb, mivel több lidar sugár érkezik vissza, képernyőfelvételek

File: urdf/mecanum.xacro (robot description, xacro)
@@ -2,9 +2,9 @@
 <robot xmlns:xacro="https://www.ros.org/wiki/xacro" name="mecanum" xmlns:ignition="http://gazebosim.org/schema">
 <!-- <xacro:include filename="hokuyo_ust10.xacro" /> -->
-<xacro:property name="radius" value="0.065" />
-<xacro:property name="length" value="0.08" />
-<xacro:property name="box_length" value="0.5" />
-<xacro:property name="box_width" value="0.3" />
-<xacro:property name="box_height" value="0.1" />
+<xacro:property name="radius" value="0.05" />
+<xacro:property name="length" value="0.06" />
+<xacro:property name="box_length" value="0.3" />
+<xacro:property name="box_width" value="0.2" />
+<xacro:property name="box_height" value="0.09" />
 <material name="blue">
  <color rgba="0 0 0.8 1" />
@@ -23,5 +23,5 @@
         <origin xyz="0 0 0" rpy="1.57075 0 0"  />
         <geometry>
-            <mesh filename="file://$(find mecanum_simulation_github)/meshes/Mecanum_jo.stl" scale="0.0015 0.0015 0.0015" />
+            <mesh filename="file://$(find mecanum_simulation_github)/meshes/Mecanum_jo.stl" scale="0.0010 0.0010 0.0010" />
         </geometry>
         <material name="black" />
@@ -41,5 +41,5 @@
     <parent link="base_link" />
     <child link="front_right_wheel" />
-    <origin xyz="0.2 -${box_width/2+length/2} -0.03" />
+    <origin xyz="0.1 -${box_width/2+length/2} -0.03" />
     <axis xyz="0 1 0" />
 </joint>
@@ -48,5 +48,5 @@
         <origin xyz="0 0 0" rpy="1.57075 0 0"  />
         <geometry>
-            <mesh filename="file://$(find mecanum_simulation_github)/meshes/Mecanum_jo.stl" scale="0.0015 0.0015 0.0015" />
+            <mesh filename="file://$(find mecanum_simulation_github)/meshes/Mecanum_jo.stl" scale="0.0010 0.0010 0.0010" />
         </geometry>
         <material name="black" />
@@ -66,5 +66,5 @@
     <parent link="base_link" />
     <child link="front_left_wheel" />
-    <origin xyz="0.2 ${box_width/2+length/2} -0.03" />
+    <origin xyz="0.1 ${box_width/2+length/2} -0.03" />
     <axis xyz="0 1 0" />
 </joint>
@@ -73,5 +73,5 @@
         <origin xyz="0 0 0" rpy="1.57075 0 0"  />
         <geometry>
-            <mesh filename="file://$(find mecanum_simulation_github)/meshes/Mecanum_jo.stl" scale="0.0015 0.0015 0.0015" />
+            <mesh filename="file://$(find mecanum_simulation_github)/meshes/Mecanum_jo.stl" scale="0.0010 0.0010 0.0010" />
         </geometry>
         <material name="black" />
@@ -91,5 +91,5 @@
     <parent link="base_link" />
     <child link="rear_left_wheel" />
-    <origin xyz="-0.2 ${box_width/2+length/2} -0.03" />
+    <origin xyz="-0.1 ${box_width/2+length/2} -0.03" />
     <axis xyz="0 1 0" />
 </joint>
@@ -98,5 +98,5 @@
         <origin xyz="0 0 0" rpy="1.57075 0 0"  />
         <geometry>
-            <mesh filename="file://$(find mecanum_simulation_github)/meshes/Mecanum_jo.stl" scale="0.0015 0.0015 0.0015" />
+            <mesh filename="file://$(find mecanum_simulation_github)/meshes/Mecanum_jo.stl" scale="0.0010 0.0010 0.0010" />
         </geometry>
         <material name="black" />
@@ -116,5 +116,5 @@
     <parent link="base_link" />
     <child link="rear_right_wheel" />
-    <origin xyz="-0.2 -${box_width/2+length/2} -0.03" />
+    <origin xyz="-0.1 -${box_width/2+length/2} -0.03" />
     <axis xyz="0 1 0" />
 </joint>
@@ -149,5 +149,5 @@
         <origin xyz="0 0 -0.05" rpy="0 0 3.14"  />
         <geometry>
-            <mesh filename="file://$(find mecanum_simulation_github)/meshes/sensors/hokuyo_ust10.stl" scale="1 1 1" />
+            <mesh filename="file://$(find mecanum_simulation_github)/meshes/sensors/hokuyo_ust10.stl" scale="0.8 0.8 0.8" />
         </geometry>
         <material name="white" />
@@ -168,9 +168,9 @@
     <parent link="base_link" />
     <child link="base_scan" />
-    <origin xyz="0.175 0 0.1" rpy="0 0 3.1415" />
+    <origin xyz="0.1 0 0.09" rpy="0 0 0" />
 </joint>
 <gazebo reference="base_scan">
 <sensor name="base_scan" type="gpu_lidar">
-        <pose>0 0 0 0 0 0</pose>
+        <pose relative_to='base_scan'>0 0 0 0 0 0</pose>
         <topic>scan</topic>
         <gz_frame_id>base_scan</gz_frame_id>
@@ -179,21 +179,21 @@
           <scan>
             <horizontal>
-              <samples>1200</samples>
-              <resolution>0.8</resolution>
+              <samples>500</samples>
+              <resolution>1</resolution>
               <min_angle>0</min_angle>
               <max_angle>6.28</max_angle>
-              <angle_increment>0.0175</angle_increment>
+              <!-- <angle_increment>0.0175</angle_increment> -->
             </horizontal>
-            <vertical>
+            <!-- <vertical>
               <samples>1</samples>
               <resolution>1</resolution>
               <min_angle>0</min_angle>
               <max_angle>0</max_angle>
-            </vertical>
+            </vertical> -->
           </scan>
           <range>
             <min>0.120</min>
             <max>10.0</max>
-            <resolution>0.015</resolution>
+            <resolution>0.25</resolution>
           </range>
           <noise>

Commit message: lidar szenzor 270 fok, jó irányban áll a csatlakozó, tesztelve GAZEBO-ban, RVIZ-ben

File: urdf/mecanum.xacro (robot description, xacro)
@@ -147,5 +147,5 @@
 <link name="base_scan">
     <visual>
-        <origin xyz="0 0 -0.05" rpy="0 0 3.14"  />
+        <origin xyz="0 0 -0.05" rpy="0 0 0"  />
         <geometry>
             <mesh filename="file://$(find mecanum_simulation_github)/meshes/sensors/hokuyo_ust10.stl" scale="0.8 0.8 0.8" />
@@ -181,6 +181,6 @@
               <samples>500</samples>
               <resolution>1</resolution>
-              <min_angle>0</min_angle>
-              <max_angle>6.28</max_angle>
+              <min_angle>-2.3562</min_angle>
+              <max_angle>2.3562</max_angle>
               <!-- <angle_increment>0.0175</angle_increment> -->
             </horizontal>

Commit message: inerciák kiszámolva, lidar fekete gazebo-ban és rvizben is, tesztelve mindkát szoftverben

File: urdf/mecanum.xacro (robot description, xacro)
@@ -4,7 +4,9 @@
 <xacro:property name="radius" value="0.05" />
 <xacro:property name="length" value="0.06" />
+<xacro:property name="mass" value="0.4" />
 <xacro:property name="box_length" value="0.3" />
 <xacro:property name="box_width" value="0.2" />
 <xacro:property name="box_height" value="0.09" />
+<xacro:property name="box_mass" value="3.0" />
 <material name="blue">
  <color rgba="0 0 0.8 1" />
@@ -34,6 +36,6 @@
     </collision>
     <inertial>
-        <mass value="0.3"/>
-        <inertia ixx="1e-3" ixy="0" ixz="0" iyy="1e-3" iyz="0" izz="1e-3" />
+        <mass value="${mass}"/>
+        <inertia ixx="${1/12*mass*(3*radius*radius+length*length)}" ixy="0" ixz="0" iyy="${1/2*mass*radius*radius}" iyz="0" izz="${1/12*mass*(3*radius*radius+length*length)}" />
     </inertial>
 </link>
@@ -59,6 +61,6 @@
     </collision>
     <inertial>
-        <mass value="0.3"/>
-        <inertia ixx="1e-3" ixy="0" ixz="0" iyy="1e-3" iyz="0" izz="1e-3" />
+        <mass value="${mass}"/>
+        <inertia ixx="${1/12*mass*(3*radius*radius+length*length)}" ixy="0" ixz="0" iyy="${1/2*mass*radius*radius}" iyz="0" izz="${1/12*mass*(3*radius*radius+length*length)}" />
     </inertial>
 </link>
@@ -84,6 +86,6 @@
     </collision>
     <inertial>
-        <mass value="0.3"/>
-        <inertia ixx="1e-3" ixy="0" ixz="0" iyy="1e-3" iyz="0" izz="1e-3" />
+        <mass value="${mass}"/>
+        <inertia ixx="${1/12*mass*(3*radius*radius+length*length)}" ixy="0" ixz="0" iyy="${1/2*mass*radius*radius}" iyz="0" izz="${1/12*mass*(3*radius*radius+length*length)}" />
     </inertial>
 </link>
@@ -109,6 +111,6 @@
     </collision>
     <inertial>
-        <mass value="0.3"/>
-        <inertia ixx="1e-3" ixy="0" ixz="0" iyy="1e-3" iyz="0" izz="1e-3" />
+        <mass value="${mass}"/>
+        <inertia ixx="${1/12*mass*(3*radius*radius+length*length)}" ixy="0" ixz="0" iyy="${1/2*mass*radius*radius}" iyz="0" izz="${1/12*mass*(3*radius*radius+length*length)}" />
     </inertial>
 </link>
@@ -135,6 +137,6 @@
     <inertial>
         <origin xyz="-0.02 0 0.035" rpy="0 0 0" />
-        <mass value="3.0" />
-        <inertia ixx="0.0300" ixy="0" ixz="0" iyy="0.1" iyz="0" izz="0.1" />
+        <mass value="${box_mass}" />
+        <inertia ixx="${1/12*box_mass*(box_height*box_height+box_width*box_width)}" ixy="0" ixz="0" iyy="${1/12*box_mass*(box_length*box_length+box_height*box_height)}" iyz="0" izz="${1/12*box_mass*(box_length*box_length+box_width*box_width)}" />
     </inertial>
 </link>
@@ -151,5 +153,5 @@
             <mesh filename="file://$(find mecanum_simulation_github)/meshes/sensors/hokuyo_ust10.stl" scale="0.8 0.8 0.8" />
         </geometry>
-        <material name="white" />
+        <material name="black" />
     </visual>
     <collision>
@@ -207,4 +209,5 @@
         <visualize>true</visualize>
       </sensor>
+    <material>Gazebo/Black</material>
 </gazebo>
 <!-- <gazebo>

Commit message: Diplomaterv_B nem tudom hol tartottam

File: urdf/mecanum.xacro (robot description, xacro)
@@ -3,5 +3,5 @@
 <!-- <xacro:include filename="hokuyo_ust10.xacro" /> -->
 <xacro:property name="radius" value="0.05" />
-<xacro:property name="length" value="0.06" />
+<xacro:property name="length" value="0.05" />
 <xacro:property name="mass" value="0.4" />
 <xacro:property name="box_length" value="0.3" />
@@ -196,5 +196,5 @@
           <range>
             <min>0.120</min>
-            <max>10.0</max>
+            <max>20.0</max>
             <resolution>0.25</resolution>
           </range>

Commit message: Robotkar mesh RVIZ-ben és Gazebo-ban is megjelenik, elhelyezést pontosítani kell még

File: urdf/mecanum.xacro (robot description, xacro)
@@ -21,4 +21,7 @@
  <color rgba="1 1 1 1" />
 </material>
+<material name="orange">
+ <color rgba="1 0.5 0 1" />
+</material>
 <link name="front_right_wheel">
     <visual>
@@ -171,4 +174,179 @@
     <child link="base_scan" />
     <origin xyz="0.1 0 0.09" rpy="0 0 0" />
+</joint>
+<link name="link_0">
+    <visual>
+        <origin xyz="0 0 0" rpy="1.57075 0 0"  />
+        <geometry>
+            <mesh filename="file://$(find mecanum_simulation_github)/meshes/simplify_link_0.stl" scale="0.0003 0.0003 0.0003" />
+        </geometry>
+        <material name="orange" />
+    </visual>
+    <collision>
+        <origin xyz="0 0 0" rpy="0 0 0"  />
+        <geometry>
+            <cylinder length="${length}" radius="${radius}" />
+        </geometry>
+    </collision>
+    <inertial>
+        <mass value="${mass}"/>
+        <inertia ixx="${1/12*mass*(3*radius*radius+length*length)}" ixy="0" ixz="0" iyy="${1/2*mass*radius*radius}" iyz="0" izz="${1/12*mass*(3*radius*radius+length*length)}" />
+    </inertial>
+</link>
+<joint name="teto" type="fixed">
+    <parent link="base_link" />
+    <child link="link_0" />
+    <origin xyz="-0.02 0 0.05" />
+    <axis xyz="0 1 0" />
+</joint>
+<link name="link_1">
+    <visual>
+        <origin xyz="0 0 0" rpy="1.57075 0 0"  />
+        <geometry>
+            <mesh filename="file://$(find mecanum_simulation_github)/meshes/simplify_link_1.stl" scale="0.0003 0.0003 0.0003" />
+        </geometry>
+        <material name="orange" />
+    </visual>
+    <collision>
+        <origin xyz="0 0 0" rpy="0 0 0"  />
+        <geometry>
+            <cylinder length="${length}" radius="${radius}" />
+        </geometry>
+    </collision>
+    <inertial>
+        <mass value="${mass}"/>
+        <inertia ixx="${1/12*mass*(3*radius*radius+length*length)}" ixy="0" ixz="0" iyy="${1/2*mass*radius*radius}" iyz="0" izz="${1/12*mass*(3*radius*radius+length*length)}" />
+    </inertial>
+</link>
+<joint name="rob_joint_1" type="fixed">
+    <parent link="link_0" />
+    <child link="link_1" />
+    <origin xyz="-0.02 0 0.05" />
+    <axis xyz="0 1 0" />
+</joint>
+<link name="link_2">
+    <visual>
+        <origin xyz="0 0 0" rpy="1.57075 0 0"  />
+        <geometry>
+            <mesh filename="file://$(find mecanum_simulation_github)/meshes/simplify_link_2.stl" scale="0.0003 0.0003 0.0003" />
+        </geometry>
+        <material name="orange" />
+    </visual>
+    <collision>
+        <origin xyz="0 0 0" rpy="0 0 0"  />
+        <geometry>
+            <cylinder length="${length}" radius="${radius}" />
+        </geometry>
+    </collision>
+    <inertial>
+        <mass value="${mass}"/>
+        <inertia ixx="${1/12*mass*(3*radius*radius+length*length)}" ixy="0" ixz="0" iyy="${1/2*mass*radius*radius}" iyz="0" izz="${1/12*mass*(3*radius*radius+length*length)}" />
+    </inertial>
+</link>
+<joint name="rob_joint_2" type="fixed">
+    <parent link="link_1" />
+    <child link="link_2" />
+    <origin xyz="-0.02 0 0.05" />
+    <axis xyz="0 1 0" />
+</joint>
+<link name="link_3">
+    <visual>
+        <origin xyz="0 0 0" rpy="1.57075 0 0"  />
+        <geometry>
+            <mesh filename="file://$(find mecanum_simulation_github)/meshes/simplify_link_3.stl" scale="0.0003 0.0003 0.0003" />
+        </geometry>
+        <material name="orange" />
+    </visual>
+    <collision>
+        <origin xyz="0 0 0" rpy="0 0 0"  />
+        <geometry>
+            <cylinder length="${length}" radius="${radius}" />
+        </geometry>
+    </collision>
+    <inertial>
+        <mass value="${mass}"/>
+        <inertia ixx="${1/12*mass*(3*radius*radius+length*length)}" ixy="0" ixz="0" iyy="${1/2*mass*radius*radius}" iyz="0" izz="${1/12*mass*(3*radius*radius+length*length)}" />
+    </inertial>
+</link>
+<joint name="rob_joint_3" type="fixed">
+    <parent link="link_2" />
+    <child link="link_3" />
+    <origin xyz="-0.02 0 0.05" />
+    <axis xyz="0 1 0" />
+</joint>
+<link name="link_4">
+    <visual>
+        <origin xyz="0 0 0" rpy="1.57075 0 0"  />
+        <geometry>
+            <mesh filename="file://$(find mecanum_simulation_github)/meshes/simplify_link_4.stl" scale="0.0003 0.0003 0.0003" />
+        </geometry>
+        <material name="orange" />
+    </visual>
+    <collision>
+        <origin xyz="0 0 0" rpy="0 0 0"  />
+        <geometry>
+            <cylinder length="${length}" radius="${radius}" />
+        </geometry>
+    </collision>
+    <inertial>
+        <mass value="${mass}"/>
+        <inertia ixx="${1/12*mass*(3*radius*radius+length*length)}" ixy="0" ixz="0" iyy="${1/2*mass*radius*radius}" iyz="0" izz="${1/12*mass*(3*radius*radius+length*length)}" />
+    </inertial>
+</link>
+<joint name="rob_joint_4" type="fixed">
+    <parent link="link_3" />
+    <child link="link_4" />
+    <origin xyz="-0.02 0 0.05" />
+    <axis xyz="0 1 0" />
+</joint>
+<link name="link_5">
+    <visual>
+        <origin xyz="0 0 0" rpy="1.57075 0 0"  />
+        <geometry>
+            <mesh filename="file://$(find mecanum_simulation_github)/meshes/simplify_link_5.stl" scale="0.0003 0.0003 0.0003" />
+        </geometry>
+        <material name="orange" />
+    </visual>
+    <collision>
+        <origin xyz="0 0 0" rpy="0 0 0"  />
+        <geometry>
+            <cylinder length="${length}" radius="${radius}" />
+        </geometry>
+    </collision>
+    <inertial>
+        <mass value="${mass}"/>
+        <inertia ixx="${1/12*mass*(3*radius*radius+length*length)}" ixy="0" ixz="0" iyy="${1/2*mass*radius*radius}" iyz="0" izz="${1/12*mass*(3*radius*radius+length*length)}" />
+    </inertial>
+</link>
+<joint name="rob_joint_5" type="fixed">
+    <parent link="link_4" />
+    <child link="link_5" />
+    <origin xyz="-0.02 0 0.05" />
+    <axis xyz="0 1 0" />
+</joint>
+<link name="link_6">
+    <visual>
+        <origin xyz="0 0 0" rpy="1.57075 0 0"  />
+        <geometry>
+            <mesh filename="file://$(find mecanum_simulation_github)/meshes/simplify_link_6.stl" scale="0.0003 0.0003 0.0003" />
+        </geometry>
+        <material name="orange" />
+    </visual>
+    <collision>
+        <origin xyz="0 0 0" rpy="0 0 0"  />
+        <geometry>
+            <cylinder length="${length}" radius="${radius}" />
+        </geometry>
+    </collision>
+    <inertial>
+        <mass value="${mass}"/>
+        <inertia ixx="${1/12*mass*(3*radius*radius+length*length)}" ixy="0" ixz="0" iyy="${1/2*mass*radius*radius}" iyz="0" izz="${1/12*mass*(3*radius*radius+length*length)}" />
+    </inertial>
+</link>
+<joint name="rob_joint_6" type="fixed">
+    <parent link="link_5" />
+    <child link="link_6" />
+    <origin xyz="-0.02 0 0.05" />
+    <axis xyz="0 1 0" />
 </joint>
 <gazebo reference="base_scan">
@@ -340,3 +518,8 @@
     <mu2>0.000002</mu2>
   </gazebo>
+  <gazebo reference="link_0">
+    <material>Gazebo/Orange</material>
+    <mu1>0.000002</mu1>
+    <mu2>0.000002</mu2>
+  </gazebo>
 </robot>

Commit message: urdf-ben a 0-2 link jól van pozícionálva

File: urdf/mecanum.xacro (robot description, xacro)
@@ -177,9 +177,9 @@
 <link name="link_0">
     <visual>
-        <origin xyz="0 0 0" rpy="1.57075 0 0"  />
+        <origin xyz="-0.005 0.010 -0.035" rpy="1.57075 0 0"  />
         <geometry>
             <mesh filename="file://$(find mecanum_simulation_github)/meshes/simplify_link_0.stl" scale="0.0003 0.0003 0.0003" />
         </geometry>
-        <material name="orange" />
+        <material name="yellow" />
     </visual>
     <collision>
@@ -197,14 +197,14 @@
     <parent link="base_link" />
     <child link="link_0" />
-    <origin xyz="-0.02 0 0.05" />
+    <origin xyz="-0.02 0.0075 0.080" />
     <axis xyz="0 1 0" />
 </joint>
 <link name="link_1">
     <visual>
-        <origin xyz="0 0 0" rpy="1.57075 0 0"  />
-        <geometry>
-            <mesh filename="file://$(find mecanum_simulation_github)/meshes/simplify_link_1.stl" scale="0.0003 0.0003 0.0003" />
-        </geometry>
-        <material name="orange" />
+        <origin xyz="-0.020 -0.030 -0.005" rpy="1.57075 0 0"  />
+        <geometry>
+            <mesh filename="file://$(find mecanum_simulation_github)/meshes/simplify_link_1.stl" scale="-0.0003 0.0003 0.0003" />
+        </geometry>
+        <material name="blue" />
     </visual>
     <collision>
@@ -222,14 +222,14 @@
     <parent link="link_0" />
     <child link="link_1" />
-    <origin xyz="-0.02 0 0.05" />
-    <axis xyz="0 1 0" />
+    <origin xyz="0 0 0" rpy="0 0 0"/>
+    <axis xyz="0 0 1" />
 </joint>
 <link name="link_2">
     <visual>
-        <origin xyz="0 0 0" rpy="1.57075 0 0"  />
-        <geometry>
-            <mesh filename="file://$(find mecanum_simulation_github)/meshes/simplify_link_2.stl" scale="0.0003 0.0003 0.0003" />
-        </geometry>
-        <material name="orange" />
+        <origin xyz="0.01 -0.045 -0.025" rpy="1.57075 0 0"  />
+        <geometry>
+            <mesh filename="file://$(find mecanum_simulation_github)/meshes/simplify_link_2.stl" scale="-0.0003 0.0003 0.0003" />
+        </geometry>
+        <material name="yellow" />
     </visual>
     <collision>
@@ -247,5 +247,5 @@
     <parent link="link_1" />
     <child link="link_2" />
-    <origin xyz="-0.02 0 0.05" />
+    <origin xyz="0.01 0 0.07" />
     <axis xyz="0 1 0" />
 </joint>
@@ -272,5 +272,5 @@
     <parent link="link_2" />
     <child link="link_3" />
-    <origin xyz="-0.02 0 0.05" />
+    <origin xyz="-0.02 0 1" />
     <axis xyz="0 1 0" />
 </joint>
@@ -297,5 +297,5 @@
     <parent link="link_3" />
     <child link="link_4" />
-    <origin xyz="-0.02 0 0.05" />
+    <origin xyz="-0.02 0 1" />
     <axis xyz="0 1 0" />
 </joint>
@@ -322,5 +322,5 @@
     <parent link="link_4" />
     <child link="link_5" />
-    <origin xyz="-0.02 0 0.05" />
+    <origin xyz="-0.02 0 1" />
     <axis xyz="0 1 0" />
 </joint>
@@ -347,5 +347,5 @@
     <parent link="link_5" />
     <child link="link_6" />
-    <origin xyz="-0.02 0 0.05" />
+    <origin xyz="-0.02 0 1" />
     <axis xyz="0 1 0" />
 </joint>
